File: breakout_pcb/nea_fixture_breakout_board.sch (KiCad schematic (older format))
At the start: 30 parts, among them P1 CONN_02X13, P2 CONN_02X15, U1 MS8607

Commit message: -updated schematic with unique resistor values at each sensor location -created pdfs of the schematic and pcb layout
Parts:
- R10: value 10k -> 6.81k; description (none) -> RES SMD 1K OHM 1% 1/10W 0603; manufacturer (none) -> Yageo; manufacturer pn (none) -> RC0603FR-071KL; supplier (none) -> digikey; supplier pn (none) -> 311-1.00KHRCT-ND
- R11: value 10k -> 7.5k; description (none) -> RES SMD 1K OHM 1% 1/10W 0603; manufacturer (none) -> Yageo; manufacturer pn (none) -> RC0603FR-071KL; supplier (none) -> digikey; supplier pn (none) -> 311-1.00KHRCT-ND
- R12: value 10k -> 8.2k; description (none) -> RES SMD 1K OHM 1% 1/10W 0603; manufacturer (none) -> Yageo; manufacturer pn (none) -> RC0603FR-071KL; supplier (none) -> digikey; supplier pn (none) -> 311-1.00KHRCT-ND
- R13: description (none) -> RES SMD 1K OHM 1% 1/10W 0603; manufacturer (none) -> Yageo; manufacturer pn (none) -> RC0603FR-071KL; supplier (none) -> digikey; supplier pn (none) -> 311-1.00KHRCT-ND
- R14: value 10k -> 11k; description (none) -> RES SMD 1K OHM 1% 1/10W 0603; manufacturer (none) -> Yageo; manufacturer pn (none) -> RC0603FR-071KL; supplier (none) -> digikey; supplier pn (none) -> 311-1.00KHRCT-ND
- R15: value 10k -> 12k; description (none) -> RES SMD 1K OHM 1% 1/10W 0603; manufacturer (none) -> Yageo; manufacturer pn (none) -> RC0603FR-071KL; supplier (none) -> digikey; supplier pn (none) -> 311-1.00KHRCT-ND
- R16: value 10k -> 13k; description (none) -> RES SMD 1K OHM 1% 1/10W 0603; manufacturer (none) -> Yageo; manufacturer pn (none) -> RC0603FR-071KL; supplier (none) -> digikey; supplier pn (none) -> 311-1.00KHRCT-ND
- R17: value 10k -> 14k; description (none) -> RES SMD 1K OHM 1% 1/10W 0603; manufacturer (none) -> Yageo; manufacturer pn (none) -> RC0603FR-071KL; supplier (none) -> digikey; supplier pn (none) -> 311-1.00KHRCT-ND
- R18: value 10k -> 15k; description (none) -> RES SMD 1K OHM 1% 1/10W 0603; manufacturer (none) -> Yageo; manufacturer pn (none) -> RC0603FR-071KL; supplier (none) -> digikey; supplier pn (none) -> 311-1.00KHRCT-ND
- R19: value 10k -> 16k; description (none) -> RES SMD 1K OHM 1% 1/10W 0603; manufacturer (none) -> Yageo; manufacturer pn (none) -> RC0603FR-071KL; supplier (none) -> digikey; supplier pn (none) -> 311-1.00KHRCT-ND
- R2: value 10k -> 1.5k; description (none) -> RES SMD 1.5K OHM 1% 1/10W 0603; manufacturer (none) -> Yageo; manufacturer pn (none) -> RC0603FR-071K5L; supplier (none) -> digikey; supplier pn (none) -> 311-1.50KHRCT-ND
- R20: value 10k -> 17.4k; description (none) -> RES SMD 1K OHM 1% 1/10W 0603; manufacturer (none) -> Yageo; manufacturer pn (none) -> RC0603FR-071KL; supplier (none) -> digikey; supplier pn (none) -> 311-1.00KHRCT-ND
- R21: value 10k -> 18k; description (none) -> RES SMD 1K OHM 1% 1/10W 0603; manufacturer (none) -> Yageo; manufacturer pn (none) -> RC0603FR-071KL; supplier (none) -> digikey; supplier pn (none) -> 311-1.00KHRCT-ND
- R22: value 10k -> 20k; description (none) -> RES SMD 1K OHM 1% 1/10W 0603; manufacturer (none) -> Yageo; manufacturer pn (none) -> RC0603FR-071KL; supplier (none) -> digikey; supplier pn (none) -> 311-1.00KHRCT-ND
- R3: value 10k -> 2k; description (none) -> RES SMD 1K OHM 1% 1/10W 0603; manufacturer (none) -> Yageo; manufacturer pn (none) -> RC0603FR-071KL; supplier (none) -> digikey; supplier pn (none) -> 311-1.00KHRCT-ND
- R4: value 10k -> 2.7k; description (none) -> RES SMD 1K OHM 1% 1/10W 0603; manufacturer (none) -> Yageo; manufacturer pn (none) -> RC0603FR-071KL; supplier (none) -> digikey; supplier pn (none) -> 311-1.00KHRCT-ND
- R5: value 10k -> 3.3k; description (none) -> RES SMD 1K OHM 1% 1/10W 0603; manufacturer (none) -> Yageo; manufacturer pn (none) -> RC0603FR-071KL; supplier (none) -> digikey; supplier pn (none) -> 311-1.00KHRCT-ND
- R6: value 10k -> 3.9k; description (none) -> RES SMD 1K OHM 1% 1/10W 0603; manufacturer (none) -> Yageo; manufacturer pn (none) -> RC0603FR-071KL; supplier (none) -> digikey; supplier pn (none) -> 311-1.00KHRCT-ND
- R7: value 10k -> 4.7k; description (none) -> RES SMD 1K OHM 1% 1/10W 0603; manufacturer (none) -> Yageo; manufacturer pn (none) -> RC0603FR-071KL; supplier (none) -> digikey; supplier pn (none) -> 311-1.00KHRCT-ND
- R8: value 10k -> 5.6k; description (none) -> RES SMD 1K OHM 1% 1/10W 0603; manufacturer (none) -> Yageo; manufacturer pn (none) -> RC0603FR-071KL; supplier (none) -> digikey; supplier pn (none) -> 311-1.00KHRCT-ND
- R9: value 10k -> 6.2k; description (none) -> RES SMD 1K OHM 1% 1/10W 0603; manufacturer (none) -> Yageo; manufacturer pn (none) -> RC0603FR-071KL; supplier (none) -> digikey; supplier pn (none) -> 311-1.00KHRCT-ND
- U1: symbol MS8607 -> MS8607-RESCUE-nea_fixture_breakout_board
