File: pcb-breakout/nea_fixture_breakout_board.sch (KiCad schematic (older format))
At the start: 30 parts, among them P1 CONN_02X13, P2 CONN_02X15, U1 MS8607

Commit message: --fixed breakout pcb drill file for reorder and regenerated gerbers --
Parts:
- added H3: dowel_holes2, footprints_on_Cdrive:dowel_holes2, symbol dowel_holes
- added R23, R24: 10k, Resistors_SMD:R_0603_HandSoldering, symbol Res1
Connections:
- wire segments 130 -> 135
Changed lines of the file:
@@
 	6250 5000 6690 5000
 Wire Wire Line
-	2800 5650 2380 5650
+	2290 5650 2800 5650
 Wire Wire Line
 	2800 5850 2380 5850
@@
 	4020 5650 3600 5650
 Wire Wire Line
-	4020 5750 3600 5750
+	3600 5750 4300 5750
 Text Label 2380 5650 0    60   ~ 0
 VDD
@@
 NoConn ~ 2800 5950
 $Comp
-L GND #PWR4
+L GND #PWR01
 U 1 1 58872187
 P 2380 5930
-F 0 "#PWR4" H 2380 5680 50  0001 C CNN
+F 0 "#PWR01" H 2380 5680 50  0001 C CNN
 F 1 "GND" H 2380 5780 50  0000 C CNN
 F 2 "" H 2380 5930 50  0000 C CNN
@@
 LED2
 $Comp
-L GND #PWR1
+L GND #PWR02
 U 1 1 5887396D
 P 6690 5085
-F 0 "#PWR1" H 6690 4835 50  0001 C CNN
+F 0 "#PWR02" H 6690 4835 50  0001 C CNN
 F 1 "GND" H 6690 4935 50  0000 C CNN
 F 2 "" H 6690 5085 50  0000 C CNN
@@
 	7350 4800 7350 5230
 $Comp
-L GND #PWR3
+L GND #PWR03
 U 1 1 58875A11
 P 7350 5740
-F 0 "#PWR3" H 7350 5490 50  0001 C CNN
+F 0 "#PWR03" H 7350 5490 50  0001 C CNN
 F 1 "GND" H 7350 5590 50  0000 C CNN
 F 2 "" H 7350 5740 50  0000 C CNN
@@
 	5750 4800 5330 4800
 $Comp
-L GND #PWR2
+L GND #PWR04
 U 1 1 5888F80B
 P 4950 5535
-F 0 "#PWR2" H 4950 5285 50  0001 C CNN
+F 0 "#PWR04" H 4950 5285 50  0001 C CNN
 F 1 "GND" H 4950 5385 50  0000 C CNN
 F 2 "" H 4950 5535 50  0000 C CNN
@@
 	0    1    1    0
 $EndComp
+$Comp
+L Res1 R24
+U 1 1 5892A783
+P 4300 5390
+F 0 "R24" H 4420 5415 40  0000 C CNN
+F 1 "10k" H 4425 5340 40  0000 C CNN
+F 2 "Resistors_SMD:R_0603_HandSoldering" H 4230 5390 30  0001 C CNN
+F 3 "" H 4300 5390 30  0000 C CNN
+F 4 "digikey" V 4300 5390 60  0001 C CNN "supplier"
+F 5 "311-1.00KHRCT-ND" V 4300 5390 60  0001 C CNN "supplier pn"
+F 6 "Yageo" V 4300 5390 60  0001 C CNN "manufacturer"
+F 7 " RC0603FR-071KL " V 4300 5390 60  0001 C CNN "manufacturer pn"
+F 8 " RES SMD 1K OHM 1% 1/10W 0603 " V 4300 5390 60  0001 C CNN "description"
+	1    4300 5390
+	1    0    0    -1
+$EndComp
+$Comp
+L Res1 R23
+U 1 1 5892AEA4
+P 4020 5385
+F 0 "R23" H 4140 5405 40  0000 C CNN
+F 1 "10k" H 4140 5330 40  0000 C CNN
+F 2 "Resistors_SMD:R_0603_HandSoldering" H 3950 5385 30  0001 C CNN
+F 3 "" H 4020 5385 30  0000 C CNN
+F 4 "digikey" V 4020 5385 60  0001 C CNN "supplier"
+F 5 "311-1.00KHRCT-ND" V 4020 5385 60  0001 C CNN "supplier pn"
+F 6 "Yageo" V 4020 5385 60  0001 C CNN "manufacturer"
+F 7 " RC0603FR-071KL " V 4020 5385 60  0001 C CNN "manufacturer pn"
+F 8 " RES SMD 1K OHM 1% 1/10W 0603 " V 4020 5385 60  0001 C CNN "description"
+	1    4020 5385
+	1    0    0    -1
+$EndComp
+Wire Wire Line
+	4020 5650 4020 5510
+Wire Wire Line
+	4300 5750 4300 5515
+Text Label 4020 5020 0    60   ~ 0
+VDD
+Wire Wire Line
+	4300 5290 4300 5190
+Wire Wire Line
+	4300 5190 4020 5190
+Wire Wire Line
+	4020 5020 4020 5285
+Connection ~ 4020 5190
+$Comp
+L dowel_holes H3
+U 1 1 589314F8
+P 4385 7410
+F 0 "H3" H 4380 7490 60  0000 C CNN
+F 1 "dowel_holes2" H 4405 7385 60  0000 C CNN
+F 2 "footprints_on_Cdrive:dowel_holes2" H 4385 7410 118 0001 C CNN
+F 3 "" H 4385 7410 118 0000 C CNN
+	1    4385 7410
+	1    0    0    -1
+$EndComp
 $EndSCHEMATC
