File: pcb-measurement_circuits/nea_research_pcb_rev1.sch (KiCad schematic (older format))
At the start: 102 parts, among them U1 TPS73125, U10 AD5144, U11 GasSensor8x2-CLCC36, U12 TLV1G125, U13 TPS73133, U14 AD8603, U15 TLV1G125, U16 AD5144, U17 AD5144, U18 AD8603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

Commit message: --fixed breakout pcb drill file for reorder and regenerated gerbers --
Parts:
- added P4, P5: CONN_02X05, Pin_Headers:Pin_Header_Straight_2x05_Pitch2.54mm, symbol CONN_02X05
- P2: renamed from P?; footprint Footprints:header_smt_2x15 -> Pin_Headers:Pin_Header_Straight_2x15_Pitch2.54mm
- P3: renamed from P?; footprint Footprints:header_smt_2x13 -> Pin_Headers:Pin_Header_Straight_2x13_Pitch2.54mm
- gave numbers to parts that had none: 4
Connections:
- net labels added: 5V, STROBE
- net labels removed: 12V, VIN
- wire segments 484 -> 497
Other:
- note added: "DATA CONNECTORS"
- note added: "DATA IN"
- note added: "DATA OUT"
- moved on the sheet: C1, C10, C11, C12, C13, C14, C15, C17, C19, C2, C21, C22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
