File: pcb-switch_board/backups/nea_research_pcb_rev1_switch.kicad_pcb (KiCad board)
At the start: 2 copper layers, 100 x 50 mm, 8 parts, among them P1 CONN_02X15, P2 CONN_02X13, P3 CONN_02X30, U1 QS4A110, U2 QS4A110, U3 QS4A110, U4 QS4A110, U5 QS4A110

Commit message: -laying out switch board
Parts:
- moved U1 4.72 mm to (-17.3, -12.8)
- moved U2 0.48 mm to (-13.5, 1.07)
Connections:
- U1 pad 15: (no net) -> /B2_SW
- U1 pad 5: /B2_SW -> /MID2_SW
- U2 pad 15: (no net) -> /G2_SW
- U2 pad 5: /G2_SW -> /E2_SW
- U3 pad 15: (no net) -> /L2_SW
- U4 pad 15: (no net) -> /Q2_SW
- U4 pad 5: /Q2_SW -> /O2_SW
- U5 pad 15: (no net) -> /V2_SW
Routing:
- net /MID2: track 0.00 -> 43.3 mm, vias 0 -> 1
- net /B2_SW: track 0.00 -> 18.0 mm
- net /C1_SW: track 0.00 -> 16.6 mm
- net /B1_SW: track 0.00 -> 14.6 mm
- net /C2_SW: track 0.00 -> 13.8 mm
- net /A2_SW: track 0.00 -> 13.6 mm
- net /D1_SW: track 0.00 -> 12.7 mm
- net /A1_SW: track 0.00 -> 11.5 mm
- net /MID2_SW: track 0.00 -> 9.51 mm
- net /D2_SW: track 0.00 -> 9.51 mm
- net /MID1: track 12.3 -> 3.21 mm, vias 0 -> 1
- net /B1: track 11.9 -> 3.41 mm, vias 0 -> 1
- net /A1: track 12.1 -> 4.04 mm, vias 0 -> 1
- net /D2: track 8.50 -> 16.3 mm, vias 0 -> 3
- net /MID1_SW: track 0.00 -> 7.36 mm
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