File: pcb-breakout/rev2/nea_fixture_breakout_board_rev2.kicad_pcb (KiCad board)
At the start: 2 copper layers, 60 x 40 mm, 38 parts, among them P1 CONN_02X13, P2 CONN_02X15, U1 BME280

Commit message: -removed solder paste layer from breakout board bond pad footprint -starting on control board schematic
Parts:
- U1: footprint footprints_on_Cdrive:BME280 -> footprints_on_Cdrive:BME280_hand
