File: pcb-control_board/_saved_nea_research_control_board.sch (KiCad schematic (older format))
At the start: 18 parts, among them P1 Rpi_HDR-40, P2 CONN_02X30, U1 AD7683, U2 ADG706, U3 ADG706, U4 ADG706, U5 ADG706, U6 ADG706, U7 ADG706, U8 TPS73133

Commit message: -updated wiring diagram for breakout board and switch board headers -fixed switch board schematic pdf naming
Parts:
- added C? (x5): 0.1uF, footprints_on_Cdrive:0402, symbol CAP_NP
- added C?: 10uF, footprints_on_Cdrive:0402, symbol CAP_NP
- added D1: LED_SMT, footprints:0603-D, symbol LED_SMT
- added R2: 75, footprints_on_Cdrive:0603, symbol Res1_1
- added R?: 1K, footprints_on_Cdrive:0402, symbol Res1_1
- added U? (x4): 74LS08, symbol 74LS08
- added U?: MCP4921, footprints_on_Cdrive:, symbol MCP4921
Connections:
- net labels added: DAC_CS, DAC_OUT, SIMO_SDA, SPI_CLK, V2P5, gnd_mux_en, ~ADC_CS
- net labels removed: ADC_CS, CLK_SW, V1P25, ~CS_SW
- wire segments 285 -> 323
- no-connect marks 24 -> 25
Other:
- note added: "spare"

Commit message: -changed die_holder_block depth from 41mm to 40mm -added a probe block that is a one-piece design thick enough to hold spring probes
Parts:
- removed C? (x3): 0.1uF, footprints_on_Cdrive:0402, symbol CAP_NP
- added C10, C11, C12, C13, C7, C8, C9: 0.1uF, Resistors_SMD:R_0603_HandSoldering, symbol CAP_NP
- added P3: CONN_02X05, symbol CONN_02X05
- C1, C2: footprint footprints_on_Cdrive:0402 -> Resistors_SMD:R_0603_HandSoldering; description CAP CER 0.1UF 16V X5R 0402 -> CAP CER 0.1UF 16V X7R 0603; manufacturer pn 0402YD104KAT2A -> GRM188R71C104KA01D; supplier pn 478-1126-1-ND -> 490-1532-1-ND
- D1: Value2 (none) -> Yellow LED; description LED 1.6X0.8MM 568NM GRN CLR SMD -> LED YELLOW CLEAR 0603 SMD; manufacturer pn APT1608SGC -> APT1608LSYCK/J3-PRV; supplier pn 754-1121-1-ND -> 754-1932-1-ND
- R2: value 75 -> 1.5K; description RES SMD 75 OHM 1% 1/10W 0603 -> RES SMD 1.5K OHM 1% 1/10W 0603; manufacturer pn RC0603FR-0775RL -> RC0603FR-071K5L; supplier pn 311-75.0HRCT-ND -> 311-1.50KHRCT-ND
- U9: renamed from U?; footprint (none) -> footprints_on_Cdrive:SOIC-14_N; description (none) -> IC GATE AND 4CH 2-INP 14-SO; manufacturer (none) -> Diodes Inc.; manufacturer pn (none) -> 74HC08S14-13; supplier (none) -> digikey; supplier pn (none) -> 74HC08S14-13DICT-ND
- gave numbers to parts that had none: 6
Connections:
- net labels added: 5V_OUT, GPIO12, GPIO16, GPIO20, GPIO21, GPIO22, GPIO24, GPIO25, GPIO5, GPIO6, ~DAC_CS
- net labels removed: DAC_CS
- wire segments 323 -> 356
- no-connect marks 25 -> 27
Other:
- note added: "Bypass Caps"
- moved on the sheet: C4, C5, C6, D1, P1, R2, TP1, U8
