File: pcb-measurement board/_saved_measurement_board.sch (KiCad schematic (older format))
At the start: 76 parts, among them P1 CONN_02X15, P2 CONN_02X13, P3 HDR DUAL ROW, P4 CONN_02X05, P5 CONN_02X05, Q2 Si1101X, U1 TPS73125, U10 AD8603, U11 TLV1G125, U12 MCP4921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

Commit message: -schematic is being refined -working on placement of pcb parts -all footprints are completed
Parts:
- added R13: 18k, footprints_on_Cdrive:0402, symbol Res1_1
- added R16: DNI, footprints_on_Cdrive:0603, symbol Res1_1
- R1: value 1K -> ?; footprint footprints_on_Cdrive:0402 -> footprints_on_Cdrive:0603; description RES SMD 1K OHM 1% 1/16W 0402 -> (none); manufacturer pn RC0402FR-071KL -> (none); supplier pn 311-1.00KLRCT-ND -> (none)
- R10: value 1K -> DNI; footprint footprints_on_Cdrive:0402 -> footprints_on_Cdrive:0603; description RES SMD 1K OHM 1% 1/16W 0402 -> (none); manufacturer Yageo -> (none); manufacturer pn RC0402FR-071KL -> (none); supplier digikey -> (none); supplier pn 311-1.00KLRCT-ND -> (none)
- R2: value 10K -> ?; footprint footprints_on_Cdrive:0402 -> footprints_on_Cdrive:0603; description RES SMD 10K OHM 1% 1/16W 0402 -> (none); manufacturer pn RC0402FR-0710KL -> (none); supplier pn 311-10.0KLRCT-ND -> (none)
- R5: value 100K -> ?; footprint footprints_on_Cdrive:0402 -> footprints_on_Cdrive:0603; description RES SMD 100K OHM 1% 1/16W 0402 -> (none); manufacturer Stackpole Electronics Inc. -> Yageo; manufacturer pn RC0402FR-07100KL -> (none); supplier pn 311-100KLRCT-ND -> (none)
- R6: value 1M -> ?; footprint footprints_on_Cdrive:0402 -> footprints_on_Cdrive:0603; description RES SMD 1M OHM 1% 1/16W 0402 -> (none); manufacturer Stackpole Electronics Inc. -> Yageo; manufacturer pn RC0402FR-071ML -> (none); supplier pn 311-1.00MLRCT-ND -> (none)
- R8: value 1K -> 100k; description RES SMD 1K OHM 1% 1/16W 0402 -> RES SMD 100K OHM 1% 1/16W 0402; manufacturer Yageo -> Stackpole Electronics Inc.; manufacturer pn RC0402FR-071KL -> RC0402FR-07100KL; supplier pn 311-1.00KLRCT-ND -> 311-100KLRCT-ND
- U16: footprint (none) -> footprints_on_Cdrive:SOT23-8
- gave numbers to parts that had none: 2
Connections:
- net labels added: 0V5, ~SELG
- net labels removed: SELG
- wire segments 476 -> 481
Other:
- moved on the sheet: C27
